File: kicad/keyatura/keyatura.kicad_pcb (KiCad board)
At the start: 2 copper layers, 256.5 x 126.2 mm, 82 parts, among them J1 Battery, SW1 SW_Push, SW10 SW_Push, SW11 SW_Push, SW12 SW_Push, SW13 SW_Push, SW14 SW_Push, SW15 SW_Push, SW16 SW_Push, SW17 SW_Push, SW18 SW_Push, SW19 SW_Push, SW2 SW_Push, SW20 SW_Push, SW21 SW_Push, SW22 SW_Push, SW23 SW_Push, SW24 SW_Push, SW25 SW_Push, SW26 SW_Push, SW27 SW_Push, SW28 SW_Push, SW29 SW_Push, SW3 SW_Push, SW30 SW_Push, SW31 SW_Push, SW32 SW_Push, SW33 SW_Push, SW34 SW_Push, SW35 SW_Push, SW36 SW_Push, SW4 SW_Push, SW5 SW_Push, SW6 SW_Push, SW7 SW_Push, SW8 SW_Push, SW9 SW_Push, U1 SuperMini nRF52840

Commit message: added gerber files
Parts:
- added G*** (x3): LOGO, LOGO, F.Cu at (239.7, 103.6)
- added H0: MountingHole, keyatura:mounting hole, F.Cu at (44.7, 96.8)
- added H1: MountingHole, keyatura:mounting hole, B.Cu at (264.0, 96.0)
- added H2: MountingHole, keyatura:mounting hole, F.Cu at (180.0, 51.1)
- added H3: MountingHole, keyatura:mounting hole, F.Cu at (120.7, 41.7)
- added H4: MountingHole, keyatura:mounting hole, F.Cu at (52.9, 33.3)
- added H5: MountingHole, keyatura:mounting hole, F.Cu at (254.6, 34.4)
- added H6: MountingHole, keyatura:mounting hole, F.Cu at (176.4, 115.0)
- added H7: MountingHole, keyatura:mounting hole, F.Cu at (132.4, 115.0)
- moved L0 37.3 mm to (148.5, 84.7)
- moved L1 37.3 mm to (154.5, 84.7)
- moved L2 37.3 mm to (160.5, 84.7)
- moved R0 37.3 mm to (148.5, 87.7)
- moved R1 37.3 mm to (154.5, 87.7)
- moved R2 37.3 mm to (160.5, 87.7)
- moved J1 7.48 mm to (154.5, 91.1)
- moved RST_BTN1 3.15 mm to (154.4, 146.0), turned to 180 degrees
- moved BAT_KEY1 2.30 mm to (154.4, 135.2)
Connections:
- U1 pad 1: C4 -> C0
- U1 pad 2: C3 -> C1
- U1 pad 6: C1 -> C3
- U1 pad 7: C0 -> C4
Routing:
- net C0: track 0.00 -> 513.8 mm
- net C1: track 0.00 -> 452.7 mm
- net C2: track 0.00 -> 402.1 mm
- net C3: track 0.00 -> 341.9 mm
- net C4: track 0.00 -> 283.5 mm
- net R5: track 0.00 -> 164.1 mm
- net R4: track 0.00 -> 135.8 mm
- net R6: track 0.00 -> 130.4 mm
- net R7: track 0.00 -> 115.8 mm
- net RST: track 0.00 -> 109.6 mm
- net BAT+: track 0.00 -> 98.5 mm
- net Net-(BAT_KEY1-B): track 0.00 -> 79.4 mm
- net R0: track 45.2 -> 121.7 mm
- net LED2: track 0.00 -> 30.6 mm
- net LED1: track 0.00 -> 27.8 mm
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- added copper zone on B.Cu, net GND
- added copper zone on F.Cu, net GND
Other:
- outline, holes or cut-outs redrawn
